File: electronics/MacroPad.kicad_sch (KiCad schematic)
At the start: 52 parts, among them SW0 SW_Coded, SW1 SW_Push, SW10 SW_Push, SW11 SW_Push, SW12 SW_Push, SW13 SW_Push, SW14 SW_Push, SW15 SW_Push, SW16 SW_Push, SW17 SW_Push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

Commit message: platformio conversion
Parts:
- added BT1: Battery, Connector_PinHeader_2.00mm:PinHeader_1x02_P2.00mm_Vertical, symbol Device:Battery
- added C1, C2: 4.7uF, Capacitor_SMD:C_0603_1608Metric_Pad1.08x0.95mm_HandSolder, symbol Device:C_Polarized
- added R2: 2K, Resistor_SMD:R_1210_3225Metric_Pad1.30x2.65mm_HandSolder, symbol Device:R
- added SW25: SW_SPDT, Connector_PinHeader_2.54mm:PinHeader_1x03_P2.54mm_Vertical, symbol Switch:SW_SPDT
- added U4: MCP73831T-2ACI_OT, proj_components:SOT95P280X145-5N, symbol MCP73831:MCP73831T-2ACI_OT
- D1, D10, D11, D12, D13, D14, D15, D16, D17, D18, D19, D2, D20, D21, D22, D23, D24, D3, D4, D5, D6, D7, D8, D9: value 1N4148 -> LL4148; footprint Diode_SMD:D_1210_3225Metric_Pad1.42x2.65mm_HandSolder -> LL4148:LL4148; symbol Diode:1N4148 -> jlcpartnumbers:LL4148; LCSC (none) -> C435829
Connections:
- net +5V: now also SW25.2 (B); no longer U2.24 (RAW)
- net GND: now also BT1.2 (-), C1.2, C2.2, R2.2, U4.2 (VSS)
- net STAT: now reaches U2.20 (D21/A3/PF4)
- net STAT: now also U4.1 (STAT)
- new net: BT1.1 (+), C2.1, SW25.1 (A), U4.3 (VBAT)
- new net: C1.1, SW25.3 (C), U4.4 (VDD)
- new net: R2.1, U4.5 (PROG)
- no-connect marks 20 -> 21
